Commit message: Fix steel frame collision issue

File: hdz_ros2_ws/src/hdz_base_description/urdf/hdz_base_macro.xacro (robot description, xacro)
@@ -145,9 +145,31 @@
             </visual>
             <collision>
-                <origin
-                    xyz="0 0 0"
-                    rpy="0 0 0" />
-                <geometry>
-                    <mesh filename="package://hdz_base_description/meshes/hdz_steel_frame_link.STL" />
+                <origin xyz="0 0.20995 0.250326" rpy="0 0 0" />
+                <geometry>
+                   <box size="0.250326 0.021692 0.503987"/>
+                </geometry>
+            </collision>
+            <collision>
+                <origin xyz="-0.132548 0 0.250326" rpy="0 0 ${radians(90)}" />
+                <geometry>
+                   <box size="0.430527 0.021692 0.503987"/>
+                </geometry>
+            </collision>
+            <collision>
+                <origin xyz="0 -0.210101 0.250326" rpy="0 0 0" />
+                <geometry>
+                   <box size="0.250326 0.021692 0.503987"/>
+                </geometry>
+            </collision>
+            <collision>
+                <origin xyz="0 0 0.493123" rpy="${radians(90)} 0 0" />
+                <geometry>
+                   <box size="0.286785 0.025388 0.44325"/>
+                </geometry>
+            </collision>
+            <collision>
+                <origin xyz="0.00297 0 0.595211" rpy="0 0 0" />
+                <geometry>
+                   <cylinder radius="0.052649" length="0.18"/>
                 </geometry>
             </collision>
@@ -203,10 +225,9 @@
             <collision>
                 <origin
-                    xyz="0 0 0"
-                    rpy="0 0 0" />
-                <geometry>
-                    <mesh
-                        filename="package://hdz_base_description/meshes/hdz_ur_control_cabinet_link.STL" />
-                </geometry>
+                    xyz="0 0 0.05228"
+                    rpy="0 0 0" />
+               <geometry>
+                <box size="0.261088 0.383256 0.106136"/>
+               </geometry>
             </collision>
         </link>

File: hdz_ros2_ws/src/hdz_moveit_assistant/config/hdz_full.ros2_control.xacro (robot description, xacro)
@@ -2,5 +2,5 @@
 <robot xmlns:xacro="http://www.ros.org/wiki/xacro">
     <xacro:macro name="hdz_full_ros2_control" params="name initial_positions_file">
-        <xacro:property name="initial_positions" value="${load_yaml(initial_positions_file)['initial_positions']}"/>
+        <xacro:property name="initial_positions" value="${xacro.load_yaml(initial_positions_file)}"/>
         <ros2_control name="${name}" type="system">
             <hardware>

File: hdz_ros2_ws/src/hdz_moveit_assistant/config/hdz_full.urdf.xacro (robot description, xacro)
@@ -1,5 +1,5 @@
 <?xml version="1.0"?>
 <robot xmlns:xacro="http://www.ros.org/wiki/xacro" name="hdz_full">
-    <xacro:arg name="initial_positions_file" default="initial_positions.yaml" />
+    <xacro:arg name="initial_positions_file" default="$(find hdz_moveit_assistant)/config/initial_positions.yaml" />
     <!-- Import hdz_full urdf file -->
     <xacro:include filename="$(find hdz_full_description)/urdf/hdz_full.xacro" />

File: hdz_ros2_ws/src/hdz_moveit_config/srdf/hdz_macro.srdf.xacro (robot description, xacro)
@@ -124,6 +124,4 @@
     <disable_collisions link1="camera_link" link2="wrist_2_link" reason="Never"/>
     <disable_collisions link1="camera_link" link2="wrist_3_link" reason="Adjacent"/>
-    <disable_collisions link1="forearm_link" link2="hdz_steel_frame_link" reason="Default"/>
-    <disable_collisions link1="forearm_link" link2="hdz_ur_control_cabinet_link" reason="Default"/>
     <disable_collisions link1="forearm_link" link2="upper_arm_link" reason="Adjacent"/>
     <disable_collisions link1="forearm_link" link2="wrist_1_link" reason="Adjacent"/>
@@ -131,5 +129,5 @@
     <disable_collisions link1="hdz_base_link" link2="hdz_extend_board_link" reason="Adjacent"/>
     <disable_collisions link1="hdz_base_link" link2="hdz_steel_frame_link" reason="Never"/>
-    <disable_collisions link1="hdz_base_link" link2="hdz_ur_control_cabinet_link" reason="Never"/>
+    <disable_collisions link1="hdz_base_link" link2="hdz_ur_control_cabinet_link" reason="Default"/>
     <disable_collisions link1="hdz_base_link" link2="shoulder_link" reason="Never"/>
     <disable_collisions link1="hdz_extend_board_link" link2="hdz_steel_frame_link" reason="Adjacent"/>
@@ -138,7 +136,5 @@
     <disable_collisions link1="hdz_steel_frame_link" link2="hdz_ur_control_cabinet_link" reason="Adjacent"/>
     <disable_collisions link1="hdz_steel_frame_link" link2="shoulder_link" reason="Never"/>
-    <disable_collisions link1="hdz_steel_frame_link" link2="upper_arm_link" reason="Default"/>
     <disable_collisions link1="hdz_ur_control_cabinet_link" link2="shoulder_link" reason="Never"/>
-    <disable_collisions link1="hdz_ur_control_cabinet_link" link2="upper_arm_link" reason="Default"/>
     <disable_collisions link1="left_finger" link2="left_finger_pad" reason="Adjacent"/>
     <disable_collisions link1="left_finger" link2="left_inner_knuckle" reason="Default"/>

Commit message: add hdz_sim_gazebo

File: hdz_ros2_ws/src/hdz_base_description/urdf/hdz_base_macro.xacro (robot description, xacro)
@@ -2,6 +2,5 @@
 <robot xmlns:xacro="http://wiki.ros.org/xacro">
     <xacro:macro name="hdz_base_description" params="parent tf_prefix:=hdz_ *origin">
-        <link
-            name="${tf_prefix}base_link">
+        <link name="${tf_prefix}base_link">
             <inertial>
                 <origin
@@ -23,5 +22,5 @@
                     rpy="0 0 0" />
                 <geometry>
-                    <mesh filename="package://hdz_base_description/meshes/hdz_base_link.STL" />
+                    <mesh filename="file://$(find hdz_base_description)/meshes/hdz_base_link.STL" />
                 </geometry>
                 <material
@@ -37,8 +36,17 @@
                 <geometry>
                     <mesh
-                        filename="package://hdz_base_description/meshes/hdz_base_link.STL" />
-                </geometry>
-            </collision>
-        </link>
+                        filename="file://$(find hdz_base_description)/meshes/hdz_base_link.STL" />
+                </geometry>
+            </collision>
+        </link>
+        <!-- <gazebo reference="${tf_prefix}base_link">
+            <collision>
+                <surface>
+                    <contact>
+                        <collide_bitmask>0x1</collide_bitmask>
+                    </contact>
+                </surface>
+            </collision>
+        </gazebo> -->
         <!-- base_joint fixes base_link to the environment -->
         <joint name="${tf_prefix}base_joint" type="fixed">
@@ -69,5 +77,5 @@
                 <geometry>
                     <mesh
-                        filename="package://hdz_base_description/meshes/hdz_extend_board_link.STL" />
+                        filename="file://$(find hdz_base_description)/meshes/hdz_extend_board_link.STL" />
                 </geometry>
                 <material
@@ -83,5 +91,5 @@
                 <geometry>
                     <mesh
-                        filename="package://hdz_base_description/meshes/hdz_extend_board_link.STL" />
+                        filename="file://$(find hdz_base_description)/meshes/hdz_extend_board_link.STL" />
                 </geometry>
             </collision>
@@ -136,5 +144,5 @@
                 <geometry>
                     <mesh
-                        filename="package://hdz_base_description/meshes/hdz_steel_frame_link.STL" />
+                        filename="file://$(find hdz_base_description)/meshes/hdz_steel_frame_link.STL" />
                 </geometry>
                 <material
@@ -147,5 +155,5 @@
                 <origin xyz="0 0.20995 0.250326" rpy="0 0 0" />
                 <geometry>
-                   <box size="0.250326 0.021692 0.503987"/>
+                    <box size="0.250326 0.021692 0.503987" />
                 </geometry>
             </collision>
@@ -153,5 +161,5 @@
                 <origin xyz="-0.132548 0 0.250326" rpy="0 0 ${radians(90)}" />
                 <geometry>
-                   <box size="0.430527 0.021692 0.503987"/>
+                    <box size="0.430527 0.021692 0.503987" />
                 </geometry>
             </collision>
@@ -159,5 +167,5 @@
                 <origin xyz="0 -0.210101 0.250326" rpy="0 0 0" />
                 <geometry>
-                   <box size="0.250326 0.021692 0.503987"/>
+                    <box size="0.250326 0.021692 0.503987" />
                 </geometry>
             </collision>
@@ -165,5 +173,5 @@
                 <origin xyz="0 0 0.493123" rpy="${radians(90)} 0 0" />
                 <geometry>
-                   <box size="0.286785 0.025388 0.44325"/>
+                    <box size="0.286785 0.025388 0.44325" />
                 </geometry>
             </collision>
@@ -171,5 +179,5 @@
                 <origin xyz="0.00297 0 0.595211" rpy="0 0 0" />
                 <geometry>
-                   <cylinder radius="0.052649" length="0.18"/>
+                    <cylinder radius="0.052649" length="0.18" />
                 </geometry>
             </collision>
@@ -215,5 +223,5 @@
                 <geometry>
                     <mesh
-                        filename="package://hdz_base_description/meshes/hdz_ur_control_cabinet_link.STL" />
+                        filename="file://$(find hdz_base_description)/meshes/hdz_ur_control_cabinet_link.STL" />
                 </geometry>
                 <material
@@ -227,7 +235,7 @@
                     xyz="0 0 0.05228"
                     rpy="0 0 0" />
-               <geometry>
-                <box size="0.261088 0.383256 0.106136"/>
-               </geometry>
+                <geometry>
+                    <box size="0.261088 0.383256 0.106136" />
+                </geometry>
             </collision>
         </link>

File: hdz_ros2_ws/src/hdz_full_description/urdf/dh_ag95_gripper.xacro (robot description, xacro)
@@ -20,4 +20,5 @@
         use_mock_hardware="$(arg use_fake_hardware)"
         mock_sensor_commands="$(arg fake_sensor_commands)"
+        sim_gazebo="$(arg sim_gazebo)"
     />
 </robot>

File: hdz_ros2_ws/src/hdz_full_description/urdf/hdz_full.xacro (robot description, xacro)
@@ -3,4 +3,5 @@
     <xacro:arg name="use_fake_hardware" default="false" />
     <xacro:arg name="fake_sensor_commands" default="false" />
+    <xacro:arg name="sim_gazebo" default="false" />
     <!-- The "world" link -->
     <link name="world" />
@@ -9,5 +10,5 @@
     <xacro:include filename="$(find hdz_base_description)/urdf/hdz_base_macro.xacro" />
     <xacro:hdz_base_description parent="world" tf_prefix="hdz_">
-        <origin xyz="0 0 0" rpy="0 0 0" />
+        <origin xyz="0 0 0.05" rpy="0 0 0" />
     </xacro:hdz_base_description>
     <!-- UR arm -->

File: hdz_ros2_ws/src/third_party/dh_ag95_gripper_ros2/dh_ag95_description/urdf/dh_ag95_macro.xacro (robot description, xacro)
@@ -29,5 +29,5 @@
           <origin xyz="-0.036673 0.00875 -0.098336" rpy="0 0 0" />
           <geometry>
-            <mesh filename="package://dh_ag95_description/meshes/visual/outer_knuckle.stl"
+            <mesh filename="file://$(find dh_ag95_description)/meshes/visual/outer_knuckle.stl"
               scale="0.001 0.001 0.001" />
           </geometry>
@@ -39,5 +39,5 @@
           <origin xyz="-0.036673 0.00875 -0.098336" rpy="0 0 0" />
           <geometry>
-            <mesh filename="package://dh_ag95_description/meshes/collision/outer_knuckle.stl"
+            <mesh filename="file://$(find dh_ag95_description)/meshes/collision/outer_knuckle.stl"
               scale="0.001 0.001 0.001" />
           </geometry>
@@ -60,5 +60,5 @@
           <origin xyz="-0.016 0.0254 -0.10586" rpy="0 0 0" />
           <geometry>
-            <mesh filename="package://dh_ag95_description/meshes/visual/inner_knuckle.stl"
+            <mesh filename="file://$(find dh_ag95_description)/meshes/visual/inner_knuckle.stl"
               scale="0.001 0.001 0.001" />
           </geometry>
@@ -70,5 +70,5 @@
           <origin xyz="-0.016 0.0254 -0.10586" rpy="0 0 0" />
           <geometry>
-            <mesh filename="package://dh_ag95_description/meshes/collision/inner_knuckle.stl"
+            <mesh filename="file://$(find dh_ag95_description)/meshes/collision/inner_knuckle.stl"
               scale="0.001 0.001 0.001" />
           </geometry>
@@ -91,5 +91,5 @@
           <origin xyz="-0.091673 0.00875 -0.098336" rpy="0 0 0" />
           <geometry>
-            <mesh filename="package://dh_ag95_description/meshes/visual/finger.stl"
+            <mesh filename="file://$(find dh_ag95_description)/meshes/visual/finger.stl"
               scale="0.001 0.001 0.001" />
           </geometry>
@@ -101,5 +101,5 @@
           <origin xyz="-0.091673 0.00875 -0.098336" rpy="0 0 0" />
           <geometry>
-            <mesh filename="package://dh_ag95_description/meshes/collision/finger.stl"
+            <mesh filename="file://$(find dh_ag95_description)/meshes/collision/finger.stl"
               scale="0.001 0.001 0.001" />
           </geometry>
@@ -124,5 +124,5 @@
           <origin xyz="-0.0705 -0.0 -0.12056" rpy="0 0 0" />
           <geometry>
-            <mesh filename="package://dh_ag95_description/meshes/visual/finger_pad.stl"
+            <mesh filename="file://$(find dh_ag95_description)/meshes/visual/finger_pad.stl"
               scale="0.001 0.001 0.001" />
           </geometry>
@@ -134,5 +134,5 @@
           <origin xyz="-0.0705 -0.0 -0.12056" rpy="0 0 0" />
           <geometry>
-            <mesh filename="package://dh_ag95_description/meshes/collision/finger_pad.stl"
+            <mesh filename="file://$(find dh_ag95_description)/meshes/collision/finger_pad.stl"
               scale="0.001 0.001 0.001" />
           </geometry>
@@ -215,5 +215,5 @@
         <origin xyz="0 0 0" rpy="0 0 0" />
         <geometry>
-          <mesh filename="package://dh_ag95_description/meshes/visual/base_link.stl"
+          <mesh filename="file://$(find dh_ag95_description)/meshes/visual/base_link.stl"
             scale="0.001 0.001 0.001" />
         </geometry>
@@ -225,5 +225,5 @@
         <origin xyz="0 0 0" rpy="0 0 0" />
         <geometry>
-          <mesh filename="package://dh_ag95_description/meshes/collision/base_link.stl"
+          <mesh filename="file://$(find dh_ag95_description)/meshes/collision/base_link.stl"
             scale="0.001 0.001 0.001" />
         </geometry>
@@ -245,5 +245,5 @@
         <origin xyz="0.0405 0.0143 -0.0147" rpy="0 0 0" />
         <geometry>
-          <mesh filename="package://dh_ag95_description/meshes/visual/gripper_body.stl"
+          <mesh filename="file://$(find dh_ag95_description)/meshes/visual/gripper_body.stl"
             scale="0.001 0.001 0.001" />
         </geometry>
@@ -255,5 +255,5 @@
         <origin xyz="0.0405 0.0143 -0.0147" rpy="0 0 0" />
         <geometry>
-          <mesh filename="package://dh_ag95_description/meshes/collision/gripper_body.stl"
+          <mesh filename="file://$(find dh_ag95_description)/meshes/collision/gripper_body.stl"
             scale="0.001 0.001 0.001" />
         </geometry>

File: hdz_ros2_ws/src/third_party/dh_ag95_gripper_ros2/dh_gripper_driver/urdf/dh_ag95.ros2_control.xacro (robot description, xacro)
@@ -2,7 +2,10 @@
 <robot xmlns:xacro="http://www.ros.org/wiki/xacro">
     <xacro:macro name="dh_ag95_gripper_ros2_control"
-        params="name prefix com_port:=/dev/ttyUSB0 use_mock_hardware:=false mock_sensor_commands:=false">
+        params="name prefix com_port:=/dev/ttyUSB0 use_mock_hardware:=false mock_sensor_commands:=false sim_gazebo:=false">
         <ros2_control name="${name}" type="system">
             <hardware>
+                <xacro:if value="${sim_gazebo}">
+                    <plugin>gazebo_ros2_control/GazeboSystem</plugin>
+                </xacro:if>
                 <xacro:if value="${use_mock_hardware}">
                     <!-- Mock hardware -->
@@ -41,41 +44,4 @@
                 </state_interface>
             </joint>
-            <!-- <xacro:if value="${use_mock_hardware}">
-                <joint name="${prefix}right_outer_knuckle_joint">
-                    <param name="mimic">${prefix}left_outer_knuckle_joint</param>
-                    <param name="multiplier">1</param>
-                    <command_interface name="position" />
-                    <state_interface name="position" />
-                    <state_interface name="velocity" />
-                </joint>
-                <joint name="${prefix}left_inner_knuckle_joint">
-                    <param name="mimic">${prefix}left_outer_knuckle_joint</param>
-                    <param name="multiplier">1</param>
-                    <command_interface name="position" />
-                    <state_interface name="position" />
-                    <state_interface name="velocity" />
-                </joint>
-                <joint name="${prefix}right_inner_knuckle_joint">
-                    <param name="mimic">${prefix}left_outer_knuckle_joint</param>
-                    <param name="multiplier">1</param>
-                    <command_interface name="position" />
-                    <state_interface name="position" />
-                    <state_interface name="velocity" />
-                </joint>
-                <joint name="${prefix}left_finger_joint">
-                    <param name="mimic">${prefix}left_outer_knuckle_joint</param>
-                    <param name="multiplier">1</param>
-                    <command_interface name="position" />
-                    <state_interface name="position" />
-                    <state_interface name="velocity" />
-                </joint>
-                <joint name="${prefix}right_finger_joint">
-                    <param name="mimic">${prefix}left_outer_knuckle_joint</param>
-                    <param name="multiplier">1</param>
-                    <command_interface name="position" />
-                    <state_interface name="position" />
-                    <state_interface name="velocity" />
-                </joint>
-            </xacro:if> -->
         </ros2_control>
     </xacro:macro>
