Commit message: Fix issue: gripper cannot be controlled.

File: hdz_ros2_ws/src/hdz_full_description/urdf/hdz_full.xacro (robot description, xacro)
@@ -4,4 +4,6 @@
     <xacro:arg name="fake_sensor_commands" default="false" />
     <xacro:arg name="sim_gazebo" default="false" />
+    <xacro:arg name="sim_ignition" default="false" />
+    <xacro:arg name="simulation_controllers" default="" />
     <!-- The "world" link -->
     <link name="world" />
@@ -15,10 +17,4 @@
     <xacro:arg name="ur_parent" default="$(arg hdz_tf_prefix)ur_base_link" />
     <xacro:include filename="$(find hdz_full_description)/urdf/ur5e.urdf.xacro" />
-    <!-- <link name="tool0"/>
-    <joint name="tool0_joint" type="fixed">
-        <parent link="$(arg hdz_tf_prefix)ur_base_link"/>
-        <child link="tool0"/>
-        <origin xyz="0.0 0.0 0.5" rpy="0.0 0.0 0.0"/>
-    </joint> -->
     <!-- 抓取中心 -->
     <link name="grasp_center_link" />
@@ -32,3 +28,5 @@
     <!-- d435i depth camera -->
     <xacro:include filename="$(find hdz_full_description)/urdf/d435i.xacro" />
+    <!-- Gazebo -->
+    <xacro:include filename="$(find hdz_full_description)/urdf/gazebo.xacro" />
 </robot>

File: hdz_ros2_ws/src/hdz_full_description/urdf/ur5e.urdf.xacro (robot description, xacro)
@@ -43,5 +43,4 @@
   <xacro:arg name="sim_gazebo" default="false" />
   <xacro:arg name="sim_ignition" default="false" />
-  <xacro:arg name="simulation_controllers" default="" />
   <!-- initial position for simulations (Fake Hardware, Gazebo, Ignition) -->
   <xacro:arg name="initial_positions_file" default="$(find ur_description)/config/initial_positions.yaml" />
@@ -88,24 +87,3 @@
     <origin xyz="0 0 0" rpy="0 0 0" />          <!-- position robot in the world -->
   </xacro:ur_robot>
-  <xacro:if value="$(arg sim_gazebo)">
-    <!-- Gazebo plugins -->
-    <gazebo reference="world">
-    </gazebo>
-    <gazebo>
-      <plugin filename="libgazebo_ros2_control.so" name="gazebo_ros2_control">
-        <parameters>$(arg simulation_controllers)</parameters>
-      </plugin>
-    </gazebo>
-  </xacro:if>
-  <xacro:if value="$(arg sim_ignition)">
-    <!-- Gazebo plugins -->
-    <gazebo reference="world">
-    </gazebo>
-    <gazebo>
-      <plugin filename="libign_ros2_control-system.so" name="ign_ros2_control::IgnitionROS2ControlPlugin">
-        <parameters>$(arg simulation_controllers)</parameters>
-        <controller_manager_node_name>$(arg tf_prefix)controller_manager</controller_manager_node_name>
-      </plugin>
-    </gazebo>
-  </xacro:if>
 </robot>

File: hdz_ros2_ws/src/third_party/dh_ag95_gripper_ros2/dh_ag95_description/urdf/dh_ag95_macro.xacro (robot description, xacro)
@@ -174,5 +174,5 @@
       <!-- This joint closes the kinematic loop. Since loops are not allowed in URDF, but they are
       allowed in SDF, this is an SDF fragment. -->
-      <gazebo>
+      <!-- <gazebo>
         <joint name="${prefix}${fingerprefix}_inner_knuckle_to_finger_joint" type="revolute">
           <pose> -0.020673 0 0.007524 0 0 0</pose>
@@ -184,5 +184,5 @@
           <child>${prefix}${fingerprefix}_finger</child>
         </joint>
-      </gazebo>
+      </gazebo> -->
     </xacro:macro>
     <xacro:macro name="finger_pad_joint" params="prefix fingerprefix">

File: hdz_ros2_ws/src/third_party/dh_ag95_gripper_ros2/dh_gripper_driver/urdf/dh_ag95.ros2_control.xacro (robot description, xacro)
@@ -14,15 +14,7 @@
                     <!-- <param name="state_following_offset">0.0</param> -->
                 </xacro:if>
-                <xacro:unless value="${use_mock_hardware}">
+                <xacro:unless value="${use_mock_hardware or sim_gazebo}">
                     <!-- Real hardware -->
                     <plugin>dh_gripper_driver/DHGripperHardwareInterface</plugin>
-                    <!-- Parameters for the DHGripperHardwareInterface -->
-                    <!-- <param name="gripper_closed_position">0.93</param>
-                    <param name="gripper_connect_port">${com_port}</param>
-                    <param name="gripper_id">1</param>
-                    <param name="gripper_model">AG95_MB</param>
-                    <param name="gripper_baudrate">115200</param>
-                    <param name="gripper_speed_multiplier">1.0</param>
-                    <param name="gripper_force_multiplier">0.5</param> -->
                     <param name="gripper_closed_position">0.93</param>
                     <param name="COM_port">${com_port}</param>
@@ -44,4 +36,40 @@
                 </state_interface>
             </joint>
+            <!-- Mimic joints -->
+            <joint name="${prefix}right_outer_knuckle_joint">
+                <param name="mimic">${prefix}left_outer_knuckle_joint</param>
+                <param name="multiplier">1</param>
+                <command_interface name="position" />
+                <state_interface name="position" />
+                <state_interface name="velocity" />
+            </joint>
+            <joint name="${prefix}right_inner_knuckle_joint">
+                <param name="mimic">${prefix}left_outer_knuckle_joint</param>
+                <param name="multiplier">1</param>
+                <command_interface name="position" />
+                <state_interface name="position" />
+                <state_interface name="velocity" />
+            </joint>
+            <joint name="${prefix}right_finger_joint">
+                <param name="mimic">${prefix}left_outer_knuckle_joint</param>
+                <param name="multiplier">1</param>
+                <command_interface name="position" />
+                <state_interface name="position" />
+                <state_interface name="velocity" />
+            </joint>
+            <joint name="${prefix}left_inner_knuckle_joint">
+                <param name="mimic">${prefix}left_outer_knuckle_joint</param>
+                <param name="multiplier">1</param>
+                <command_interface name="position" />
+                <state_interface name="position" />
+                <state_interface name="velocity" />
+            </joint>
+            <joint name="${prefix}left_finger_joint">
+                <param name="mimic">${prefix}left_outer_knuckle_joint</param>
+                <param name="multiplier">1</param>
+                <command_interface name="position" />
+                <state_interface name="position" />
+                <state_interface name="velocity" />
+            </joint>
         </ros2_control>
     </xacro:macro>
