Commit message: Add effort interface for gazebo

File: hdz_ros2_ws/src/third_party/dh_ag95_gripper_ros2/dh_gripper_driver/urdf/dh_ag95.ros2_control.xacro (robot description, xacro)
@@ -32,44 +32,47 @@
                     <param name="initial_value">0</param>
                 </state_interface>
-                <state_interface name="velocity">
-                    <param name="initial_value">0</param>
-                </state_interface>
+                <state_interface name="velocity" />
+                <xacro:if value="${sim_gazebo}">
+                    <state_interface name="effort" />
+                </xacro:if>
             </joint>
-            <!-- Mimic joints -->
-            <joint name="${prefix}right_outer_knuckle_joint">
-                <param name="mimic">${prefix}left_outer_knuckle_joint</param>
-                <param name="multiplier">1</param>
-                <command_interface name="position" />
-                <state_interface name="position" />
-                <state_interface name="velocity" />
-            </joint>
-            <joint name="${prefix}right_inner_knuckle_joint">
-                <param name="mimic">${prefix}left_outer_knuckle_joint</param>
-                <param name="multiplier">1</param>
-                <command_interface name="position" />
-                <state_interface name="position" />
-                <state_interface name="velocity" />
-            </joint>
-            <joint name="${prefix}right_finger_joint">
-                <param name="mimic">${prefix}left_outer_knuckle_joint</param>
-                <param name="multiplier">1</param>
-                <command_interface name="position" />
-                <state_interface name="position" />
-                <state_interface name="velocity" />
-            </joint>
-            <joint name="${prefix}left_inner_knuckle_joint">
-                <param name="mimic">${prefix}left_outer_knuckle_joint</param>
-                <param name="multiplier">1</param>
-                <command_interface name="position" />
-                <state_interface name="position" />
-                <state_interface name="velocity" />
-            </joint>
-            <joint name="${prefix}left_finger_joint">
-                <param name="mimic">${prefix}left_outer_knuckle_joint</param>
-                <param name="multiplier">1</param>
-                <command_interface name="position" />
-                <state_interface name="position" />
-                <state_interface name="velocity" />
-            </joint>
+            <xacro:if value="${sim_gazebo}">
+                <!-- Mimic joints -->
+                <joint name="${prefix}right_outer_knuckle_joint">
+                    <param name="mimic">${prefix}left_outer_knuckle_joint</param>
+                    <param name="multiplier">1</param>
+                    <state_interface name="position" />
+                    <state_interface name="velocity" />
+                    <state_interface name="effort" />
+                </joint>
+                <joint name="${prefix}right_inner_knuckle_joint">
+                    <param name="mimic">${prefix}left_outer_knuckle_joint</param>
+                    <param name="multiplier">1</param>
+                    <state_interface name="position" />
+                    <state_interface name="velocity" />
+                    <state_interface name="effort" />
+                </joint>
+                <joint name="${prefix}right_finger_joint">
+                    <param name="mimic">${prefix}left_outer_knuckle_joint</param>
+                    <param name="multiplier">1</param>
+                    <state_interface name="position" />
+                    <state_interface name="velocity" />
+                    <state_interface name="effort" />
+                </joint>
+                <joint name="${prefix}left_inner_knuckle_joint">
+                    <param name="mimic">${prefix}left_outer_knuckle_joint</param>
+                    <param name="multiplier">1</param>
+                    <state_interface name="position" />
+                    <state_interface name="velocity" />
+                    <state_interface name="effort" />
+                </joint>
+                <joint name="${prefix}left_finger_joint">
+                    <param name="mimic">${prefix}left_outer_knuckle_joint</param>
+                    <param name="multiplier">1</param>
+                    <state_interface name="position" />
+                    <state_interface name="velocity" />
+                    <state_interface name="effort" />
+                </joint>
+            </xacro:if>
         </ros2_control>
     </xacro:macro>
